File: Electronics/kimble-robotti.sch (KiCad schematic (older format))
At the start: 8 parts

Commit message: Elektroniikkasuunnittelua jatkettu
Parts:
- added C? (x2): 1000uF, symbol CP
- added J?: Vacuum Pump, symbol Conn_02x01_Row_Letter_Last
- added J?: Solenoid Valve (NC), symbol Conn_02x01_Row_Letter_Last
- added J?: theta-stepper, symbol Conn_01x04
- added J? (x2): r-stepper, symbol Conn_01x04
- added RLY?: Relay Module, digikey-footprints:Relay_JSM1-12V-5, symbol JSM1-12V-5
- added SW?: Pause-button, symbol SWITCH_PUSHBUTTON
- added SW?: Resume-button, symbol SWITCH_PUSHBUTTON
- added U?: TLE4906L, pth-semi:PG-SSO-3-02, symbol TLE4906L
Connections:
- net +12V: now also U?.23 (VIN), C?.1, RLY?.1 (COM)
- net +5V: now also U?.2 (VIO), U?.2 (VIO), U?.2 (VIO), C?.1
- net GND: now also U?.9 (EN), U?.9 (EN), U?.9 (EN), C?.2, C?.2, J?.1b (Pin_1b), J?.1b (Pin_1b), RLY?.2 (COIL), SW?.1 (A), SW?.1 (A), U?.2 (GND)
- net at U?.26 (5V): now also U?.1 (V+)
- net at U?.3 (2): now also U?.3 (Vout)
- net at U?.6 (PWM-5): now also U?.13 (MISO-12)
- net at U?.7 (PWM-6): now also U?.11 (SS-PWM-10)
- net at U?.8 (7): now also U?.10 (PWM-9)
- net at U?.19 (3): now also RLY?.5 (COIL)
- net at U?.21 (1): now also SW?.2 (B)
- net at U?.22 (0): now also SW?.2 (B)
- net at U?.3 (2): now also U?.15 (STEP)
- net at U?.4 (PWM-3): now also U?.15 (STEP)
- net at U?.5 (4): now also U?.15 (STEP)
- net at U?.6 (PWM-5): now also U?.16 (DIR)
- net at U?.7 (PWM-6): now also U?.16 (DIR)
- net at U?.8 (7): now also U?.16 (DIR)
- net at U?.3 (M1B): now also J?.1 (Pin_1) (x3)
- net at U?.4 (M1A): now also J?.2 (Pin_2) (x3)
- net at U?.5 (M2A): now also J?.3 (Pin_3) (x3)
- net at U?.6 (M2B): now also J?.4 (Pin_4) (x3)
- new net: J?.1a (Pin_1a), RLY?.3 (NO)
- new net: J?.1a (Pin_1a), RLY?.4 (NC)
Other:
- note added: "Kimble-robotin elektroniikka"
- note added: "Raspberry Pi 3 on yhdistetty GRBL-Arduinoon USB:lla"
- note added: "Theta-akselin nollakohdan etsimiseen käytetään\nKimble-levyn pohjaan liimattua magneettia ja\nHall-anturia. Jos kytkin-tyyppisellä Hall-anturilla\nei päästä riittävään toistettavuuteen, voidaan käyttää\nmyös lineaarisesti riippuvaa Hall-anturia kytkemällä\nse AUX-Arduinon analogisisääntuloon."
- note added: "z-motor driver"
- note removed: "Z-motor driver"
- moved on the sheet: U?

Commit message: Kaikki osat lienee elektroniikan suunnitelmassa
Parts:
- added J?: NPT5 liikennevalo, symbol Conn_01x06
- added Q1, Q2, Q3: BC547, TO_SOT_Packages_THT:TO-92_Molded_Narrow, symbol BC547
- added R1, R2, R3: 1k2, symbol R
- added SW3: Start-button, symbol SWITCH_PUSHBUTTON
- gave numbers to parts that had none: 19
Connections:
- net +12V: now also U2.23 (VIN)
- net GND: now also J?.1 (Pin_1), J?.2 (Pin_2), Q1.3 (E), Q2.3 (E), Q3.3 (E), SW3.2 (B)
- net at J6.32 (GPIO12): now also SW3.1 (A)
- net at J6.36 (GPIO16): now also R3.2
- net at J6.38 (GPIO20): now also R1.1
- net at J6.40 (GPIO21): now also R2.2
- new net: Q3.2 (B), R2.1
- new net: Q2.2 (B), R1.2
- new net: Q1.2 (B), R3.1
- new net: J?.6 (Pin_6), Q1.1 (C)
- new net: J?.5 (Pin_5), Q2.1 (C)
- new net: J?.4 (Pin_4), Q3.1 (C)
- no-connect marks 0 -> 4
Other:
- note added: "GND"
- note added: "Keltainen"
- note added: "Logitech C920 webkamera on yhdistetty Raspberry Pi:hin USB:lla"
- note added: "Punainen"
- note added: "Vihreä"
- note added: "Vilkunta (pois)"
- note added: "Äänimerkki (päälle)"
- moved on the sheet: C1, C2, J1, J2, J3, J4, J5, J6, RLY1, SW1, SW2, U1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
